File: WandLite/WandLite.kicad_sch (KiCad schematic)
At the start: 16 parts, among them J10 VCC-O, J11 PB1-O, J12 PB0-O, J13 GND-O, J14 VCC-I, J3 PB2-MDDN, J4 Conn_01x03_Pin, J5 PB3-MDUP, J6 PB4-TRIG, J7 GND-C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

Commit message: short relief and output
Parts:
- J10, J11, J12, J13, J14, J3, J5, J6, J7, J8: footprint Connector_Wire:SolderWire-0.25sqmm_1x01_D0.65mm_OD1.7mm_Relief -> Kelvin_Library:SolderWire-0.15sqmm_1x01_D0.5mm_OD1.5mm_Relief_SHORT
Changed lines of the file:
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@@
 			)
 		)
-		(property "Footprint" "Connector_Wire:SolderWire-0.25sqmm_1x01_D0.65mm_OD1.7mm_Relief"
+		(property "Footprint" "Kelvin_Library:SolderWire-0.15sqmm_1x01_D0.5mm_OD1.5mm_Relief_SHORT"
 			(at 190.5 87.63 0)
 			(effects
@@
 			)
 		)
-		(property "Footprint" "Connector_Wire:SolderWire-0.25sqmm_1x01_D0.65mm_OD1.7mm_Relief"
+		(property "Footprint" "Kelvin_Library:SolderWire-0.15sqmm_1x01_D0.5mm_OD1.5mm_Relief_SHORT"
 			(at 101.6 92.71 0)
 			(effects
@@
 			)
 		)
-		(property "Footprint" "Connector_Wire:SolderWire-0.25sqmm_1x01_D0.65mm_OD1.7mm_Relief"
+		(property "Footprint" "Kelvin_Library:SolderWire-0.15sqmm_1x01_D0.5mm_OD1.5mm_Relief_SHORT"
 			(at 190.5 92.71 0)
 			(effects
@@
 			)
 		)
-		(property "Footprint" "Connector_Wire:SolderWire-0.25sqmm_1x01_D0.65mm_OD1.7mm_Relief"
+		(property "Footprint" "Kelvin_Library:SolderWire-0.15sqmm_1x01_D0.5mm_OD1.5mm_Relief_SHORT"
 			(at 101.6 97.79 0)
 			(effects
@@
 			)
 		)
-		(property "Footprint" "Connector_Wire:SolderWire-0.25sqmm_1x01_D0.65mm_OD1.7mm_Relief"
+		(property "Footprint" "Kelvin_Library:SolderWire-0.15sqmm_1x01_D0.5mm_OD1.5mm_Relief_SHORT"
 			(at 189.23 158.75 0)
 			(effects
@@
 			)
 		)
-		(property "Footprint" "Connector_Wire:SolderWire-0.25sqmm_1x01_D0.65mm_OD1.7mm_Relief"
+		(property "Footprint" "Kelvin_Library:SolderWire-0.15sqmm_1x01_D0.5mm_OD1.5mm_Relief_SHORT"
 			(at 101.6 100.33 0)
 			(effects
@@
 			)
 		)
-		(property "Footprint" "Connector_Wire:SolderWire-0.25sqmm_1x01_D0.65mm_OD1.7mm_Relief"
+		(property "Footprint" "Kelvin_Library:SolderWire-0.15sqmm_1x01_D0.5mm_OD1.5mm_Relief_SHORT"
 			(at 189.23 156.21 0)
 			(effects
@@
 			)
 		)
-		(property "Footprint" "Connector_Wire:SolderWire-0.25sqmm_1x01_D0.65mm_OD1.7mm_Relief"
+		(property "Footprint" "Kelvin_Library:SolderWire-0.15sqmm_1x01_D0.5mm_OD1.5mm_Relief_SHORT"
 			(at 190.5 90.17 0)
 			(effects
@@
 			)
 		)
-		(property "Footprint" "Connector_Wire:SolderWire-0.25sqmm_1x01_D0.65mm_OD1.7mm_Relief"
+		(property "Footprint" "Kelvin_Library:SolderWire-0.15sqmm_1x01_D0.5mm_OD1.5mm_Relief_SHORT"
 			(at 101.6 95.25 0)
 			(effects
@@
 			)
 		)
-		(property "Footprint" "Connector_Wire:SolderWire-0.25sqmm_1x01_D0.65mm_OD1.7mm_Relief"
+		(property "Footprint" "Kelvin_Library:SolderWire-0.15sqmm_1x01_D0.5mm_OD1.5mm_Relief_SHORT"
 			(at 190.5 85.09 0)
 			(effects
